Commit message: add vgc10 4cups type

File: onrobot_vgc10_visualization/urdf/onrobot_vgc10_1cup_model.xacro (robot description, xacro)
@@ -1,5 +1,5 @@
 <?xml version="1.0"?>
 <robot name="onrobot_vgc10_model" xmlns:xacro="http://ros.org/wiki/xacro">
-  <xacro:include filename="$(find onrobot_vgc10_visualization)/urdf/onrobot_vgc10_model_macro.xacro" />
+  <xacro:include filename="$(find onrobot_vgc10_visualization)/urdf/onrobot_vgc10_1cup_model_macro.xacro" />
   <xacro:onrobot_vgc10 prefix=""/>
 </robot>

File: onrobot_vgc10_visualization/urdf/onrobot_vgc10_1cup_model_macro.xacro (robot description, xacro)
@@ -11,5 +11,5 @@
         <origin xyz="0 0 0" rpy="0 0 0" />
         <geometry>
-          <mesh filename="package://onrobot_vgc10_visualization/meshes/visual/suction_cup.stl" />
+          <mesh filename="package://onrobot_vgc10_visualization/meshes/visual/suction_cup_1cup.stl" />
         </geometry>
         <material name="">
@@ -20,5 +20,5 @@
         <origin xyz="0 0 0" rpy="0 0 0" />
         <geometry>
-          <mesh filename="package://onrobot_vgc10_visualization/meshes/collision/suction_cup.stl" />
+          <mesh filename="package://onrobot_vgc10_visualization/meshes/collision/suction_cup_1cup.stl" />
         </geometry>
       </collision>
@@ -33,5 +33,5 @@
     </joint>
   </xacro:macro>
-  <xacro:include filename="$(find onrobot_vgc10_visualization)/urdf/onrobot_vgc10.xacro" />
+  <xacro:include filename="$(find onrobot_vgc10_visualization)/urdf/onrobot_vgc10_1cup.xacro" />
   <xacro:macro name="onrobot_vgc10" params="prefix">
     <xacro:onrobot_vgc10_base_link prefix="${prefix}"/>

File: onrobot_vgc10_visualization/urdf/onrobot_vgc10_4cups.xacro (robot description, xacro)
@@ -11,5 +11,5 @@
         <origin xyz="0 0 0" rpy="0 0 0" />
         <geometry>
-          <mesh filename="package://onrobot_vgc10_visualization/meshes/visual/base_link.stl" />
+          <mesh filename="package://onrobot_vgc10_visualization/meshes/visual/base_link_4cups.stl" />
         </geometry>
         <material name="">
@@ -20,5 +20,5 @@
         <origin xyz="0 0 0" rpy="0 0 0" />
         <geometry>
-          <mesh filename="package://onrobot_vgc10_visualization/meshes/collision/base_link.stl" />
+          <mesh filename="package://onrobot_vgc10_visualization/meshes/collision/base_link_4cups.stl" />
         </geometry>
       </collision>
