Commit message: update around gazebo

File: onrobot_rg2_description/urdf/onrobot_rg2.xacro (robot description, xacro)
@@ -30,4 +30,10 @@
         <origin xyz= "0. 0. 0." rpy="0. 0. 0." />
     </joint>
+    <gazebo reference="${prefix}onrobot_rg2_base_link">
+      <mu1>1.0</mu1>
+      <mu2>1.0</mu2>
+      <selfCollide>false</selfCollide>
+      <material>Gazebo/White</material>
+    </gazebo>
   </xacro:macro>
   <xacro:macro name="finger_joints" params="prefix fingerprefix reflect">

File: onrobot_rg2_description/urdf/onrobot_rg2_gazebo.xacro (robot description, xacro)
@@ -14,6 +14,6 @@
         <multiplier>-1.0</multiplier>
         <offset>0.0</offset>
-        <!-- <maxEffort>5.0</maxEffort>
-        <hasPID /> -->
+        <maxEffort>5.0</maxEffort>
+        <!-- <hasPID /> -->
       </plugin>
       <plugin filename="libroboticsgroup_upatras_gazebo_mimic_joint_plugin.so" name="mimic_${prefix}right_inner_knuckle_joint">
@@ -22,6 +22,6 @@
         <multiplier>-1.0</multiplier>
         <offset>0.0</offset>
-        <!-- <maxEffort>5.0</maxEffort>
-        <hasPID /> -->
+        <maxEffort>5.0</maxEffort>
+        <!-- <hasPID /> -->
       </plugin>
       <plugin filename="libroboticsgroup_upatras_gazebo_mimic_joint_plugin.so" name="mimic_${prefix}left_inner_finger_joint">
@@ -30,6 +30,6 @@
         <multiplier>1.0</multiplier>
         <offset>0.0</offset>
-        <!-- <maxEffort>5.0</maxEffort>
-        <hasPID /> -->
+        <maxEffort>5.0</maxEffort>
+        <!-- <hasPID /> -->
       </plugin>
       <plugin filename="libroboticsgroup_upatras_gazebo_mimic_joint_plugin.so" name="mimic_${prefix}right_inner_finger_joint">
@@ -38,6 +38,6 @@
         <multiplier>1.0</multiplier>
         <offset>0.0</offset>
-        <!-- <maxEffort>5.0</maxEffort>
-        <hasPID /> -->
+        <maxEffort>5.0</maxEffort>
+        <!-- <hasPID /> -->
       </plugin>
       <plugin filename="libroboticsgroup_upatras_gazebo_mimic_joint_plugin.so" name="mimic_${prefix}right_outer_knuckle_joint">
@@ -46,6 +46,6 @@
         <multiplier>-1.0</multiplier>
         <offset>0.0</offset>
-        <!-- <maxEffort>5.0</maxEffort>
-        <hasPID /> -->
+         <maxEffort>5.0</maxEffort>
+        <!-- <hasPID /> -->
       </plugin>
     </gazebo>

File: onrobot_rg2_description/urdf/onrobot_rg2_model_macro.xacro (robot description, xacro)
@@ -26,4 +26,10 @@
       </collision>
     </link>
+    <gazebo reference="${prefix}${fingerprefix}_outer_knuckle">
+      <mu1>0.1</mu1>
+      <mu2>0.1</mu2>
+      <selfCollide>false</selfCollide>
+      <material>Gazebo/White</material>
+    </gazebo>
   </xacro:macro>
   <xacro:macro name="inner_knuckle" params="prefix fingerprefix">
@@ -50,4 +56,10 @@
       </collision>
     </link>
+    <gazebo reference="${prefix}${fingerprefix}_inner_knuckle">
+      <mu1>0.1</mu1>
+      <mu2>0.1</mu2>
+      <selfCollide>false</selfCollide>
+      <material>Gazebo/White</material>
+    </gazebo>
   </xacro:macro>
   <xacro:macro name="inner_finger" params="prefix fingerprefix">
@@ -74,4 +86,13 @@
       </collision>
     </link>
+    <gazebo reference="${prefix}${fingerprefix}_inner_finger">
+      <kp>1000000.0</kp>
+      <kd>1.0</kd>
+      <mu1>1.0</mu1>
+      <mu2>1.0</mu2>
+      <minDepth>0.00001</minDepth>
+      <selfCollide>false</selfCollide>
+      <material>Gazebo/Black</material>
+    </gazebo>
   </xacro:macro>
   <xacro:macro name="inner_knuckle_joint" params="prefix fingerprefix reflect">
@@ -81,5 +102,5 @@
       <child link="${prefix}${fingerprefix}_inner_knuckle" />
       <axis xyz="1 0 0" />
-      <limit lower="-0.558505" upper="0.785398" velocity="2.0" effort="1000" />
+      <limit lower="-0.558505" upper="0.785398" velocity="100.0" effort="1000" />
       <mimic joint="${prefix}finger_joint" multiplier="-1" offset="0" />
     </joint>
@@ -91,5 +112,5 @@
       <child link="${prefix}${fingerprefix}_inner_finger" />
       <axis xyz="1 0 0" />
-      <limit lower="-0.872665" upper="0.872665" velocity="2.0" effort="1000" />
+      <limit lower="-0.872665" upper="0.872665" velocity="100.0" effort="1000" />
       <mimic joint="${prefix}finger_joint" multiplier="1" offset="0" />
     </joint>
@@ -102,5 +123,5 @@
       <child link="${prefix}left_outer_knuckle" />
       <axis xyz="-1 0 0" />
-      <limit lower="-0.558505" upper="0.785398" velocity="2.0" effort="1000" />
+      <limit lower="-0.558505" upper="0.785398" velocity="100.0" effort="1000" />
     </joint>
     <xacro:finger_joints prefix="${prefix}" fingerprefix="left" reflect="1.0"/>
@@ -112,6 +133,6 @@
       <child link="${prefix}right_outer_knuckle" />
       <axis xyz="1 0 0" />
-      <limit lower="-0.558505" upper="0.785398" velocity="2.0" effort="1000" />
-    <mimic joint="${prefix}finger_joint" multiplier="-1" offset="0" />
+      <limit lower="-0.558505" upper="0.785398" velocity="100.0" effort="1000" />
+      <mimic joint="${prefix}finger_joint" multiplier="-1" offset="0" />
     </joint>
     <xacro:finger_joints prefix="${prefix}" fingerprefix="right" reflect="-1.0"/>

File: onrobot_rg6_description/urdf/onrobot_rg6.xacro (robot description, xacro)
@@ -30,4 +30,10 @@
         <origin xyz= "0. 0. 0." rpy="0. 0. 0." />
     </joint>
+    <gazebo reference="${prefix}onrobot_rg6_base_link">
+      <mu1>1.0</mu1>
+      <mu2>1.0</mu2>
+      <selfCollide>false</selfCollide>
+      <material>Gazebo/White</material>
+    </gazebo>
   </xacro:macro>
   <xacro:macro name="finger_joints" params="prefix fingerprefix reflect">

File: onrobot_rg6_description/urdf/onrobot_rg6_gazebo.xacro (robot description, xacro)
@@ -14,6 +14,6 @@
         <multiplier>-1.0</multiplier>
         <offset>0.0</offset>
-        <!-- <maxEffort>5.0</maxEffort>
-        <hasPID /> -->
+        <maxEffort>5.0</maxEffort>
+        <!-- <hasPID /> -->
       </plugin>
       <plugin filename="libroboticsgroup_upatras_gazebo_mimic_joint_plugin.so" name="mimic_${prefix}right_inner_knuckle_joint">
@@ -22,6 +22,6 @@
         <multiplier>-1.0</multiplier>
         <offset>0.0</offset>
-        <!-- <maxEffort>5.0</maxEffort>
-        <hasPID /> -->
+        <maxEffort>5.0</maxEffort>
+        <!-- <hasPID /> -->
       </plugin>
       <plugin filename="libroboticsgroup_upatras_gazebo_mimic_joint_plugin.so" name="mimic_${prefix}left_inner_finger_joint">
@@ -30,6 +30,6 @@
         <multiplier>1.0</multiplier>
         <offset>0.0</offset>
-        <!-- <maxEffort>5.0</maxEffort>
-        <hasPID /> -->
+        <maxEffort>5.0</maxEffort>
+        <!-- <hasPID /> -->
       </plugin>
       <plugin filename="libroboticsgroup_upatras_gazebo_mimic_joint_plugin.so" name="mimic_${prefix}right_inner_finger_joint">
@@ -38,6 +38,6 @@
         <multiplier>1.0</multiplier>
         <offset>0.0</offset>
-        <!-- <maxEffort>5.0</maxEffort>
-        <hasPID /> -->
+        <maxEffort>5.0</maxEffort>
+        <!-- <hasPID /> -->
       </plugin>
       <plugin filename="libroboticsgroup_upatras_gazebo_mimic_joint_plugin.so" name="mimic_${prefix}right_outer_knuckle_joint">
@@ -46,6 +46,6 @@
         <multiplier>-1.0</multiplier>
         <offset>0.0</offset>
-        <!-- <maxEffort>5.0</maxEffort>
-        <hasPID /> -->
+        <maxEffort>5.0</maxEffort>
+        <!-- <hasPID /> -->
       </plugin>
     </gazebo>

File: onrobot_rg6_description/urdf/onrobot_rg6_model_macro.xacro (robot description, xacro)
@@ -26,4 +26,10 @@
       </collision>
     </link>
+    <gazebo reference="${prefix}${fingerprefix}_outer_knuckle">
+      <mu1>1.0</mu1>
+      <mu2>1.0</mu2>
+      <selfCollide>false</selfCollide>
+      <material>Gazebo/White</material>
+    </gazebo>
   </xacro:macro>
   <xacro:macro name="inner_knuckle" params="prefix fingerprefix">
@@ -50,4 +56,10 @@
       </collision>
     </link>
+    <gazebo reference="${prefix}${fingerprefix}_inner_knuckle">
+      <mu1>1.0</mu1>
+      <mu2>1.0</mu2>
+      <selfCollide>false</selfCollide>
+      <material>Gazebo/White</material>
+    </gazebo>
   </xacro:macro>
   <xacro:macro name="inner_finger" params="prefix fingerprefix">
@@ -74,4 +86,13 @@
       </collision>
     </link>
+    <gazebo reference="${prefix}${fingerprefix}_inner_finger">
+      <kp>1000000.0</kp>
+      <kd>1.0</kd>
+      <mu1>1.0</mu1>
+      <mu2>1.0</mu2>
+      <minDepth>0.001</minDepth>
+      <selfCollide>false</selfCollide>
+      <material>Gazebo/Black</material>
+    </gazebo>
   </xacro:macro>
   <xacro:macro name="inner_knuckle_joint" params="prefix fingerprefix reflect">
@@ -113,5 +134,5 @@
       <axis xyz="1 0 0" />
       <limit lower="-0.628319" upper="0.628319" velocity="2.0" effort="1000" />
-    <mimic joint="${prefix}finger_joint" multiplier="-1" offset="0" />
+      <mimic joint="${prefix}finger_joint" multiplier="-1" offset="0" />
     </joint>
     <xacro:finger_joints prefix="${prefix}" fingerprefix="right" reflect="-1.0"/>
