Commit message: fix a bug

File: onrobot_rg2_description/urdf/onrobot_rg2_model_macro.xacro (robot description, xacro)
@@ -89,4 +89,5 @@
       <kp>1000000.0</kp>
       <kd>1.0</kd>
+      <kd>1.0</kd>
       <mu1>1.0</mu1>
       <mu2>1.0</mu2>
@@ -102,5 +103,5 @@
       <child link="${prefix}${fingerprefix}_inner_knuckle" />
       <axis xyz="1 0 0" />
-      <limit lower="-0.558505" upper="0.785398" velocity="100.0" effort="1000" />
+      <limit lower="-0.785398" upper="0.785398" velocity="100.0" effort="1000" />
       <mimic joint="${prefix}finger_joint" multiplier="-1" offset="0" />
     </joint>
@@ -133,5 +134,5 @@
       <child link="${prefix}right_outer_knuckle" />
       <axis xyz="1 0 0" />
-      <limit lower="-0.558505" upper="0.785398" velocity="100.0" effort="1000" />
+      <limit lower="-0.785398" upper="0.785398" velocity="100.0" effort="1000" />
       <mimic joint="${prefix}finger_joint" multiplier="-1" offset="0" />
     </joint>
